File: Electronic/UI2/CursorKeypad.brd (EAGLE design)
At the start: 160 x 100 mm, 22 parts, among them IC1 74HCT14N

Commit message: new UI
Connections:
- removed net KEY: R1.1, R10.1, R2.1, R3.1, R4.1, R5.1, R6.1, R7.1, R8.1, R9.1
- removed net PULSE: IC1.10, IC1.12, IC1.2, IC1.4, IC1.8
- new net P_CENTER: IC1.8
- new net P_DOWN: IC1.4
- new net P_LEFT: IC1.12
- new net P_RIGHT: IC1.10
- new net P_UP: IC1.2
- net KEY_CENTER: now also R10.1, R9.1
- net KEY_DOWN: now also R6.1, R7.1
- net KEY_LEFT: now also R5.1, R8.1
- net KEY_RIGHT: now also R1.1, R2.1
- net KEY_UP: now also R3.1, R4.1
Changed lines of the file:
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@@
 <contactref element="KEY_LEFT" pad="P$2"/>
 <contactref element="KEY_LEFT" pad="P$1"/>
+<contactref element="R8" pad="1"/>
+<contactref element="R5" pad="1"/>
 <wire x1="38.1" y1="48.26" x2="38.1" y2="58.42" width="0" layer="19" extent="1-1"/>
+<wire x1="17.78" y1="24.13" x2="38.1" y2="48.26" width="0" layer="19" extent="1-1"/>
+<wire x1="15.24" y1="17.78" x2="17.78" y2="24.13" width="0" layer="19" extent="1-1"/>
 </signal>
 <signal name="KEY_CENTER">
 <contactref element="KEY_CENTER" pad="P$2"/>
 <contactref element="KEY_CENTER" pad="P$1"/>
+<contactref element="R9" pad="1"/>
+<contactref element="R10" pad="1"/>
+<wire x1="119.38" y1="21.59" x2="124.46" y2="29.21" width="0" layer="19" extent="1-1"/>
+<wire x1="52.07" y1="49.53" x2="119.38" y2="21.59" width="0" layer="19" extent="1-1"/>
 <wire x1="41.91" y1="49.53" x2="52.07" y2="49.53" width="0" layer="19" extent="1-1"/>
 </signal>
@@
 <contactref element="KEY_RIGHT" pad="P$2"/>
 <contactref element="KEY_RIGHT" pad="P$1"/>
+<contactref element="R2" pad="1"/>
+<contactref element="R1" pad="1"/>
 <wire x1="55.88" y1="48.26" x2="55.88" y2="58.42" width="0" layer="19" extent="1-1"/>
+<wire x1="41.91" y1="7.62" x2="55.88" y2="48.26" width="0" layer="19" extent="1-1"/>
+<wire x1="17.78" y1="8.89" x2="41.91" y2="7.62" width="0" layer="19" extent="1-1"/>
 </signal>
 <signal name="KEY_DOWN">
 <contactref element="KEY_DOWN" pad="P$2"/>
 <contactref element="KEY_DOWN" pad="P$1"/>
+<contactref element="R6" pad="1"/>
+<contactref element="R7" pad="1"/>
+<wire x1="119.38" y1="45.72" x2="124.46" y2="53.34" width="0" layer="19" extent="1-1"/>
+<wire x1="52.07" y1="36.83" x2="119.38" y2="45.72" width="0" layer="19" extent="1-1"/>
 <wire x1="41.91" y1="36.83" x2="52.07" y2="36.83" width="0" layer="19" extent="1-1"/>
 </signal>
@@
 <contactref element="KEY_UP" pad="P$2"/>
 <contactref element="KEY_UP" pad="P$1"/>
+<contactref element="R4" pad="1"/>
+<contactref element="R3" pad="1"/>
+<wire x1="52.07" y1="62.23" x2="119.38" y2="69.85" width="0" layer="19" extent="1-1"/>
 <wire x1="41.91" y1="62.23" x2="52.07" y2="62.23" width="0" layer="19" extent="1-1"/>
+<wire x1="5.08" y1="8.89" x2="41.91" y2="62.23" width="0" layer="19" extent="1-1"/>
 </signal>
 <signal name="VCC" class="1">
@@
 <wire x1="22.86" y1="17.78" x2="49.53" y2="7.62" width="0" layer="19" extent="1-1"/>
 </signal>
-<signal name="PULSE">
-<contactref element="IC1" pad="12"/>
-<contactref element="IC1" pad="10"/>
-<contactref element="IC1" pad="8"/>
-<contactref element="IC1" pad="2"/>
+<signal name="P_DOWN">
 <contactref element="IC1" pad="4"/>
-<wire x1="106.68" y1="50.8" x2="106.68" y2="55.88" width="0" layer="19" extent="1-1"/>
-<wire x1="106.68" y1="45.72" x2="106.68" y2="50.8" width="0" layer="19" extent="1-1"/>
-<wire x1="99.06" y1="58.42" x2="106.68" y2="55.88" width="0" layer="19" extent="1-1"/>
-<wire x1="99.06" y1="53.34" x2="99.06" y2="58.42" width="0" layer="19" extent="1-1"/>
 </signal>
 <signal name="K">
@@
 <wire x1="21.59" y1="41.91" x2="106.68" y2="58.42" width="0" layer="19" extent="1-1"/>
 <wire x1="25.4" y1="24.13" x2="21.59" y2="41.91" width="0" layer="19" extent="1-1"/>
-</signal>
-<signal name="KEY">
-<contactref element="R5" pad="1"/>
-<contactref element="R8" pad="1"/>
-<contactref element="R1" pad="1"/>
-<contactref element="R2" pad="1"/>
-<contactref element="R3" pad="1"/>
-<contactref element="R4" pad="1"/>
-<contactref element="R6" pad="1"/>
-<contactref element="R7" pad="1"/>
-<contactref element="R9" pad="1"/>
-<contactref element="R10" pad="1"/>
-<wire x1="124.46" y1="53.34" x2="119.38" y2="69.85" width="0" layer="19" extent="1-1"/>
-<wire x1="119.38" y1="45.72" x2="124.46" y2="53.34" width="0" layer="19" extent="1-1"/>
-<wire x1="124.46" y1="29.21" x2="119.38" y2="45.72" width="0" layer="19" extent="1-1"/>
-<wire x1="119.38" y1="21.59" x2="124.46" y2="29.21" width="0" layer="19" extent="1-1"/>
-<wire x1="41.91" y1="7.62" x2="119.38" y2="21.59" width="0" layer="19" extent="1-1"/>
-<wire x1="17.78" y1="8.89" x2="41.91" y2="7.62" width="0" layer="19" extent="1-1"/>
-<wire x1="15.24" y1="17.78" x2="17.78" y2="8.89" width="0" layer="19" extent="1-1"/>
-<wire x1="17.78" y1="24.13" x2="15.24" y2="17.78" width="0" layer="19" extent="1-1"/>
-<wire x1="5.08" y1="8.89" x2="17.78" y2="8.89" width="0" layer="19" extent="1-1"/>
 </signal>
 <signal name="K1">
@@
 <wire x1="106.68" y1="48.26" x2="119.38" y2="27.94" width="0" layer="19" extent="1-1"/>
 </signal>
+<signal name="P_LEFT">
+<contactref element="IC1" pad="12"/>
+</signal>
+<signal name="P_RIGHT">
+<contactref element="IC1" pad="10"/>
+</signal>
+<signal name="P_CENTER">
+<contactref element="IC1" pad="8"/>
+</signal>
+<signal name="P_UP">
+<contactref element="IC1" pad="2"/>
+</signal>
 </signals>

Commit message: Updated connectors
and more work on the UI Boards
Parts:
- removed C1, C2, C3, C4, C7: 1µ, rcl:C025-024X044
- removed C5: .1µ, resistor:C025-024X044
- removed IC1: 74HCT14N, 74xx-eu:DIL14
- removed R1, R3, R5, R6, R9: 82k, resistor:0204/7
- removed R10, R2, R4, R7, R8: 18k, resistor:0204/7
- added SV1: Debounce L, con-lstb:MA05-2
- added SV2: Debounce R, con-lstb:MA05-2
Connections:
- removed net K: C4.1, IC1.13, R5.2
- removed net K1: C1.1, IC1.11, R1.2
- removed net K2: C2.1, IC1.1, R3.2
- removed net K3: C3.1, IC1.3, R6.2
- removed net K4: C7.1, IC1.9, R9.2
- removed net P_CENTER: IC1.8
- removed net P_DOWN: IC1.4
- removed net P_LEFT: IC1.12
- removed net P_RIGHT: IC1.10
- removed net P_UP: IC1.2
- removed net VCC: C5.1, IC1.7, R10.2, R2.2, R4.2, R7.2, R8.2
- new net N$6: SV2.10, SV2.9
- new net N$7: SV2.7, SV2.8
- new net N$8: SV2.5, SV2.6
- new net N$9: SV2.3, SV2.4
- net GND: now also SV2.1, SV2.2; no longer C1.2, C2.2, C3.2, C4.2, C5.2, C7.2, IC1.14
- net KEY_CENTER: now also SV1.10, SV1.9; no longer R10.1, R9.1
- net KEY_DOWN: now also SV1.7, SV1.8; no longer R6.1, R7.1
- net KEY_LEFT: now also SV1.3, SV1.4; no longer R5.1, R8.1
- net KEY_RIGHT: now also SV1.1, SV1.2; no longer R1.1, R2.1
- net KEY_UP: now also SV1.5, SV1.6; no longer R3.1, R4.1
