File: Electronic/UI2/Display.sch (EAGLE design)
At the start: 6 parts, among them Q1 2N3906

Commit message: new Keycross and EC60A board
Parts:
- removed SV2: KEY_PAD, con-harting-ml:ML10L
- added C1, C10, C2, C3, C4, C5, C6, C7, C8, C9: .1µ, rcl:C-EU025-024X044
- added IC1, IC2: 74HCT14N, 74xx-eu:74HCT14N
- added IC3: 74HCT74N, 74xx-eu:74HCT74N
- added R10, R15, R4, R6, R8: 82k, resistor:R-EU_0204/7
- added R14, R3, R5, R7, R9: 15k, resistor:R-EU_0204/7
- added R16, R17, R18, R19: 10k, resistor:R-EU_0204/7
- added R20: 3k3, resistor:R-EU_0204/7
- added SV3: (no value), con-harting-ml:ML10L
Connections:
- removed net ENC-DIR: SV2.5
- removed net ENC-STEP: SV2.7
- new net ENC1: C5.1, IC2B.I, R16.2
- new net ENC2: C6.1, IC2A.I, R17.2
- new net ENC_1: R16.1, R18.1, SV3.7
- new net ENC_2: R17.1, R19.2, SV3.5
- new net K1: C9.1, IC1A.I, R14.2
- new net K2: C1.1, IC1B.I, R3.2
- new net K3: C2.1, IC1C.I, R5.2
- new net K4: C3.1, IC1E.I, R7.2
- new net K5: C4.1, IC1D.I, R9.2
- new net K_1: R14.1, R15.1, SV3.4
- new net K_2: R3.1, R4.1, SV3.6
- new net K_3: R5.1, R6.1, SV3.8
- new net K_4: R10.1, R9.1, SV3.10
- new net K_5: R7.1, R8.1, SV3.9
- new net N$1: IC2B.O, IC3A.D
- new net N$3: IC3A.CLR, IC3A.PRE, R20.2
- net !MEM_CS: now also U$1.SD_CS
- net +3.3V: now also C10.1, C7.1, C8.1, IC1P.VCC, IC2P.VCC, IC3P.VCC, R10.2, R15.2, R18.2, R19.1, R20.1, R4.2, R6.2, R8.2, SV3.1; no longer SV2.1
- net ENC_DIR: now also IC3A.Q
- net ENC_STEP: now also IC2A.O, IC3A.CLK
- net GND: now also C1.2, C10.2, C2.2, C3.2, C4.2, C5.2, C6.2, C7.2, C8.2, C9.2, IC1P.GND, IC2P.GND, IC3P.GND, SV3.2; no longer SV2.2
- net KEY_1: now also IC1A.O; no longer SV2.4
- net KEY_2: now also IC1B.O; no longer SV2.6
- net KEY_3: now also IC1C.O; no longer SV2.8
- net KEY_4: now also IC1D.O; no longer SV2.10
- net KEY_5: now also IC1E.O; no longer SV2.9
- net MISO: now also U$1.SD_MISO
- net MOSI: now also U$1.SD_MOSI
- net SCLK: now also U$1.SD_SCK
