File: Electronic/UI2/EC60_1.brd (EAGLE design)
At the start: 66 x 65.7 mm, 4 parts

Commit message: board positions
Parts:
- moved JP1 0.51 mm to (44.5, 33.1), turned to 270 degrees
- moved JP2 0.08 mm to (20.9, 33.0)
Routing:
- net GND: track 40.2 -> 0.00 mm
- net K_2: track 37.3 -> 0.00 mm
- net K_1: track 29.2 -> 0.00 mm
- net ENC_1: track 31.6 -> 40.2 mm
- net ENC_2: track 37.9 -> 44.0 mm, vias 1 -> 0
- net K_5: track 22.1 -> 26.0 mm
- net K_4: track 22.1 -> 25.3 mm
- net K_3: track 24.2 -> 25.3 mm
Changed lines of the file:
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@@
 <setting verticaltext="up"/>
 </settings>
-<grid distance="0.05" unitdist="inch" unit="mm" style="dots" multiple="1" display="no" altdistance="0.025" altunitdist="inch" altunit="mm"/>
+<grid distance="1" unitdist="mm" unit="mm" style="lines" multiple="1" display="no" altdistance="0.003125" altunitdist="mic" altunit="mm"/>
 <layers>
 <layer number="1" name="Top" color="4" fill="1" visible="yes" active="yes"/>
@@
 <class number="0" name="default" width="0" drill="0">
 </class>
-<class number="1" name="SUPPLY" width="1.016" drill="0">
+<class number="1" name="SUPPLY" width="0.254" drill="0">
 </class>
 </classes>
@@
 </autorouter>
 <elements>
-<element name="JP1" library="pinhead" package="1X03" value="" x="45.02" y="33.02" rot="R90"/>
-<element name="JP2" library="pinhead" package="1X03" value="" x="21.02" y="33.02" rot="R90"/>
+<element name="JP1" library="pinhead" package="1X03" value="" x="44.5113375" y="33.078675" rot="R270"/>
+<element name="JP2" library="pinhead" package="1X03" value="" x="20.945878125" y="33.00031875" rot="R90"/>
 <element name="SV1" library="con-harting-ml" package="ML10L" value="" x="33.02" y="50.8" rot="MR0">
 <attribute name="OC_FARNELL" value="unknown" x="33.02" y="50.8" size="1.778" layer="28" rot="MR0" display="off"/>
@@
 <contactref element="SV1" pad="2"/>
 <contactref element="JP1" pad="3"/>
-<wire x1="38.1" y1="51.435" x2="38.1" y2="52.07" width="1.016" layer="16"/>
-<wire x1="41.148" y1="48.387" x2="38.1" y2="51.435" width="1.016" layer="16"/>
-<wire x1="41.148" y1="39.37" x2="41.148" y2="48.387" width="1.016" layer="16"/>
-<wire x1="44.958" y1="35.56" x2="41.148" y2="39.37" width="1.016" layer="16"/>
-<wire x1="44.958" y1="35.56" x2="45.02" y2="35.56" width="1.016" layer="16"/>
-<wire x1="61.468" y1="41.8465" x2="63.1825" y2="41.8465" width="1.016" layer="1"/>
-<wire x1="55.1815" y1="35.56" x2="61.468" y2="41.8465" width="1.016" layer="1"/>
-<wire x1="45.02" y1="35.56" x2="55.1815" y2="35.56" width="1.016" layer="1"/>
-<wire x1="63.1825" y1="41.8465" x2="63.218" y2="41.849" width="1.016" layer="1"/>
+<wire x1="44.5113375" y1="30.538675" x2="63.218" y2="41.849" width="0" layer="19" extent="1-1"/>
+<wire x1="38.1" y1="52.07" x2="44.5113375" y2="30.538675" width="0" layer="19" extent="1-1"/>
 </signal>
 <signal name="K_1" class="1">
 <contactref element="SV1" pad="4"/>
 <contactref element="JP1" pad="2"/>
-<wire x1="36.195" y1="52.07" x2="35.56" y2="52.07" width="1.016" layer="16"/>
-<wire x1="37.592" y1="53.467" x2="36.195" y2="52.07" width="1.016" layer="16"/>
-<wire x1="39.4335" y1="53.467" x2="37.592" y2="53.467" width="1.016" layer="16"/>
-<wire x1="47.1805" y1="45.72" x2="39.4335" y2="53.467" width="1.016" layer="16"/>
-<wire x1="47.1805" y1="34.925" x2="47.1805" y2="45.72" width="1.016" layer="16"/>
-<wire x1="45.2755" y1="33.02" x2="47.1805" y2="34.925" width="1.016" layer="16"/>
-<wire x1="45.02" y1="33.02" x2="45.2755" y2="33.02" width="1.016" layer="16"/>
+<wire x1="44.5113375" y1="33.078675" x2="35.56" y2="52.07" width="0" layer="19" extent="1-1"/>
 </signal>
 <signal name="K_2" class="1">
 <contactref element="SV1" pad="6"/>
 <contactref element="JP1" pad="1"/>
-<wire x1="33.655" y1="52.07" x2="33.02" y2="52.07" width="1.016" layer="16"/>
-<wire x1="36.322" y1="54.737" x2="33.655" y2="52.07" width="1.016" layer="16"/>
-<wire x1="40.0685" y1="54.737" x2="36.322" y2="54.737" width="1.016" layer="16"/>
-<wire x1="48.3235" y1="46.482" x2="40.0685" y2="54.737" width="1.016" layer="16"/>
-<wire x1="48.3235" y1="33.528" x2="48.3235" y2="46.482" width="1.016" layer="16"/>
-<wire x1="45.2755" y1="30.48" x2="48.3235" y2="33.528" width="1.016" layer="16"/>
-<wire x1="45.02" y1="30.48" x2="45.2755" y2="30.48" width="1.016" layer="16"/>
+<wire x1="44.5113375" y1="35.618675" x2="33.02" y2="52.07" width="0" layer="19" extent="1-1"/>
 </signal>
 <signal name="K_3" class="1">
 <contactref element="SV1" pad="8"/>
 <contactref element="JP2" pad="3"/>
-<wire x1="29.845" y1="52.07" x2="30.48" y2="52.07" width="1.016" layer="1"/>
-<wire x1="28.448" y1="53.467" x2="29.845" y2="52.07" width="1.016" layer="1"/>
-<wire x1="27.432" y1="53.467" x2="28.448" y2="53.467" width="1.016" layer="1"/>
-<wire x1="24.892" y1="50.927" x2="27.432" y2="53.467" width="1.016" layer="1"/>
-<wire x1="24.892" y1="39.37" x2="24.892" y2="50.927" width="1.016" layer="1"/>
-<wire x1="21.082" y1="35.56" x2="24.892" y2="39.37" width="1.016" layer="1"/>
-<wire x1="21.082" y1="35.56" x2="21.02" y2="35.56" width="1.016" layer="1"/>
+<wire x1="20.945878125" y1="35.54031875" x2="29.21" y2="35.56" width="0.6096" layer="1"/>
+<wire x1="29.21" y1="35.56" x2="29.21" y2="50.8" width="0.6096" layer="1"/>
+<wire x1="29.21" y1="50.8" x2="30.48" y2="52.07" width="0.6096" layer="1"/>
 </signal>
 <signal name="K_4" class="1">
 <contactref element="SV1" pad="10"/>
 <contactref element="JP2" pad="2"/>
-<wire x1="27.94" y1="51.435" x2="27.94" y2="52.07" width="1.016" layer="16"/>
-<wire x1="24.892" y1="48.387" x2="27.94" y2="51.435" width="1.016" layer="16"/>
-<wire x1="24.892" y1="36.6395" x2="24.892" y2="48.387" width="1.016" layer="16"/>
-<wire x1="21.2725" y1="33.02" x2="24.892" y2="36.6395" width="1.016" layer="16"/>
-<wire x1="21.02" y1="33.02" x2="21.2725" y2="33.02" width="1.016" layer="16"/>
+<wire x1="20.945878125" y1="33.00031875" x2="26.67" y2="33.02" width="0.6096" layer="16"/>
+<wire x1="26.67" y1="33.02" x2="26.67" y2="50.8" width="0.6096" layer="16"/>
+<wire x1="26.67" y1="50.8" x2="27.94" y2="52.07" width="0.6096" layer="16"/>
 </signal>
 <signal name="K_5" class="1">
 <contactref element="SV1" pad="9"/>
 <contactref element="JP2" pad="1"/>
-<wire x1="27.94" y1="37.1475" x2="27.94" y2="49.53" width="1.016" layer="1"/>
-<wire x1="21.2725" y1="30.48" x2="27.94" y2="37.1475" width="1.016" layer="1"/>
-<wire x1="21.02" y1="30.48" x2="21.2725" y2="30.48" width="1.016" layer="1"/>
+<wire x1="27.94" y1="30.48" x2="27.94" y2="49.53" width="0.6096" layer="16"/>
+<wire x1="27.94" y1="30.48" x2="20.945878125" y2="30.46031875" width="0.6096" layer="16"/>
 </signal>
 <signal name="ENC_2" class="1">
 <contactref element="SV1" pad="7"/>
 <contactref element="U$1" pad="B"/>
-<wire x1="31.115" y1="49.53" x2="30.48" y2="49.53" width="1.016" layer="1"/>
-<wire x1="38.1635" y1="42.4815" x2="31.115" y2="49.53" width="1.016" layer="1"/>
-<wire x1="60.452" y1="42.4815" x2="38.1635" y2="42.4815" width="1.016" layer="1"/>
-<wire x1="63.3095" y1="39.624" x2="60.452" y2="42.4815" width="1.016" layer="16"/>
-<wire x1="64.262" y1="39.624" x2="63.3095" y2="39.624" width="1.016" layer="16"/>
-<wire x1="64.262" y1="39.624" x2="64.274" y2="39.584" width="1.016" layer="16"/>
-<via x="60.452" y="42.4815" extent="1-16" drill="0.3048"/>
+<wire x1="30.48" y1="49.53" x2="30.48" y2="39.37" width="0.6096" layer="1"/>
+<wire x1="30.48" y1="39.37" x2="63.5" y2="39.37" width="0.6096" layer="1"/>
+<wire x1="63.5" y1="39.37" x2="64.274" y2="39.584" width="0.6096" layer="1"/>
 </signal>
 <signal name="ENC_1" class="1">
 <contactref element="SV1" pad="5"/>
 <contactref element="U$1" pad="A"/>
-<wire x1="33.655" y1="49.53" x2="33.02" y2="49.53" width="1.016" layer="1"/>
-<wire x1="35.052" y1="48.133" x2="33.655" y2="49.53" width="1.016" layer="1"/>
-<wire x1="42.418" y1="48.133" x2="35.052" y2="48.133" width="1.016" layer="1"/>
-<wire x1="42.672" y1="48.387" x2="42.418" y2="48.133" width="1.016" layer="1"/>
-<wire x1="57.8485" y1="48.387" x2="42.672" y2="48.387" width="1.016" layer="1"/>
-<wire x1="62.103" y1="44.1325" x2="57.8485" y2="48.387" width="1.016" layer="1"/>
-<wire x1="62.103" y1="44.1325" x2="62.161" y2="44.115" width="1.016" layer="1"/>
+<wire x1="33.02" y1="41.275" x2="33.02" y2="49.53" width="0.6096" layer="1"/>
+<wire x1="33.02" y1="41.275" x2="58.42" y2="41.275" width="0.6096" layer="1"/>
+<wire x1="58.42" y1="41.275" x2="58.42" y2="43.815" width="0.6096" layer="1"/>
+<wire x1="58.42" y1="43.815" x2="62.161" y2="43.815" width="0.6096" layer="1"/>
+<wire x1="62.161" y1="43.815" x2="62.161" y2="44.115" width="0.6096" layer="1"/>
 </signal>
 <signal name="+3.3V">

Commit message: Boardwork
Parts:
- moved JP1 1.00 mm to (45.5, 33.0)
- moved JP2 0.50 mm to (20.4, 33.0)
Routing:
- net GND: track 0.00 -> 58.8 mm
- net K_1: track 0.00 -> 36.3 mm
- net K_2: track 0.00 -> 30.8 mm
Other:
- board text added: "Center"
- board text added: "GND"
Changed lines of the file:
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@@
 <setting verticaltext="up"/>
 </settings>
-<grid distance="1" unitdist="mm" unit="mm" style="lines" multiple="1" display="no" altdistance="0.003125" altunitdist="mic" altunit="mm"/>
+<grid distance="0.1" unitdist="inch" unit="mil" style="lines" multiple="1" display="yes" altdistance="0.05" altunitdist="inch" altunit="mil"/>
 <layers>
 <layer number="1" name="Top" color="4" fill="1" visible="yes" active="yes"/>
@@
 <hole x="6.02" y="6.02" drill="3.2"/>
 <hole x="60.02" y="6.02" drill="3.2"/>
+<text x="45.72" y="22.86" size="1.778" layer="25" rot="R90" align="center-left">GND</text>
+<text x="25.4" y="27.94" size="1.778" layer="25" rot="R180" align="center-left">Center</text>
 </plain>
 <attributes>
@@
 </variantdefs>
 <classes>
-<class number="0" name="default" width="0" drill="0">
+<class number="0" name="default" width="0.4064" drill="0">
 </class>
-<class number="1" name="SUPPLY" width="0.254" drill="0">
+<class number="1" name="SUPPLY" width="0.6096" drill="0">
 </class>
 </classes>
@@
 </autorouter>
 <elements>
-<element name="JP1" library="pinhead" package="1X03" value="" x="44.5113375" y="33.078675" rot="R270"/>
-<element name="JP2" library="pinhead" package="1X03" value="" x="20.945878125" y="33.00031875" rot="R90"/>
+<element name="JP1" library="pinhead" package="1X03" value="" x="45.5113375" y="33.00031875" rot="R270"/>
+<element name="JP2" library="pinhead" package="1X03" value="" x="20.445878125" y="33.00031875" rot="R90"/>
 <element name="SV1" library="con-harting-ml" package="ML10L" value="" x="33.02" y="50.8" rot="MR0">
 <attribute name="OC_FARNELL" value="unknown" x="33.02" y="50.8" size="1.778" layer="28" rot="MR0" display="off"/>
@@
 <attribute name="MF" value="" x="33.02" y="50.8" size="1.778" layer="28" rot="MR0" display="off"/>
 </element>
-<element name="U$1" library="ALPS-EC60A" package="EC60A" value="EC60A" x="33.02" y="33.02"/>
+<element name="U$1" library="ALPS-EC60A" package="EC60A" value="EC60A" x="33.000096875" y="33.00021875"/>
 </elements>
 <signals>
@@
 <contactref element="SV1" pad="2"/>
 <contactref element="JP1" pad="3"/>
-<wire x1="44.5113375" y1="30.538675" x2="63.218" y2="41.849" width="0" layer="19" extent="1-1"/>
-<wire x1="38.1" y1="52.07" x2="44.5113375" y2="30.538675" width="0" layer="19" extent="1-1"/>
+<wire x1="63.198096875" y1="41.82921875" x2="55.88" y2="41.82921875" width="0.6096" layer="16"/>
+<wire x1="55.88" y1="41.82921875" x2="36.91078125" y2="41.82921875" width="0.6096" layer="16"/>
+<wire x1="36.91078125" y1="41.82921875" x2="36.83" y2="41.91" width="0.4064" layer="16"/>
+<wire x1="36.83" y1="41.91" x2="36.83" y2="50.8" width="0.6096" layer="16"/>
+<wire x1="36.83" y1="50.8" x2="38.1" y2="52.07" width="0.6096" layer="16"/>
+<wire x1="45.5113375" y1="30.46031875" x2="55.86031875" y2="30.46031875" width="0.6096" layer="16"/>
+<wire x1="55.86031875" y1="30.46031875" x2="55.88" y2="30.48" width="0.4064" layer="16"/>
+<wire x1="55.88" y1="30.48" x2="55.88" y2="41.82921875" width="0.6096" layer="16"/>
 </signal>
 <signal name="K_1" class="1">
 <contactref element="SV1" pad="4"/>
 <contactref element="JP1" pad="2"/>
-<wire x1="44.5113375" y1="33.078675" x2="35.56" y2="52.07" width="0" layer="19" extent="1-1"/>
+<wire x1="45.5113375" y1="33.00031875" x2="46.97031875" y2="33.00031875" width="0.4064" layer="16"/>
+<wire x1="46.97031875" y1="33.00031875" x2="48.26" y2="33.02" width="0.6096" layer="16"/>
+<wire x1="48.26" y1="33.02" x2="48.26" y2="38.1" width="0.6096" layer="16"/>
+<wire x1="48.26" y1="38.1" x2="34.29" y2="38.1" width="0.6096" layer="16"/>
+<wire x1="34.29" y1="38.1" x2="34.29" y2="50.8" width="0.6096" layer="16"/>
+<wire x1="34.29" y1="50.8" x2="35.56" y2="52.07" width="0.6096" layer="16"/>
 </signal>
 <signal name="K_2" class="1">
 <contactref element="SV1" pad="6"/>
 <contactref element="JP1" pad="1"/>
-<wire x1="44.5113375" y1="35.618675" x2="33.02" y2="52.07" width="0" layer="19" extent="1-1"/>
+<wire x1="45.5113375" y1="35.54031875" x2="31.75" y2="35.54031875" width="0.6096" layer="16"/>
+<wire x1="31.75" y1="35.54031875" x2="31.75" y2="50.8" width="0.6096" layer="16"/>
+<wire x1="31.75" y1="50.8" x2="33.02" y2="52.07" width="0.6096" layer="16"/>
 </signal>
 <signal name="K_3" class="1">
 <contactref element="SV1" pad="8"/>
 <contactref element="JP2" pad="3"/>
-<wire x1="20.945878125" y1="35.54031875" x2="29.21" y2="35.56" width="0.6096" layer="1"/>
+<wire x1="20.445878125" y1="35.54031875" x2="29.21" y2="35.56" width="0.6096" layer="1"/>
 <wire x1="29.21" y1="35.56" x2="29.21" y2="50.8" width="0.6096" layer="1"/>
 <wire x1="29.21" y1="50.8" x2="30.48" y2="52.07" width="0.6096" layer="1"/>
@@
 <contactref element="SV1" pad="10"/>
 <contactref element="JP2" pad="2"/>
-<wire x1="20.945878125" y1="33.00031875" x2="26.67" y2="33.02" width="0.6096" layer="16"/>
+<wire x1="20.445878125" y1="33.00031875" x2="26.67" y2="33.02" width="0.6096" layer="16"/>
 <wire x1="26.67" y1="33.02" x2="26.67" y2="50.8" width="0.6096" layer="16"/>
 <wire x1="26.67" y1="50.8" x2="27.94" y2="52.07" width="0.6096" layer="16"/>
@@
 <contactref element="JP2" pad="1"/>
 <wire x1="27.94" y1="30.48" x2="27.94" y2="49.53" width="0.6096" layer="16"/>
-<wire x1="27.94" y1="30.48" x2="20.945878125" y2="30.46031875" width="0.6096" layer="16"/>
+<wire x1="27.94" y1="30.48" x2="20.445878125" y2="30.46031875" width="0.6096" layer="16"/>
 </signal>
 <signal name="ENC_2" class="1">
@@
 <wire x1="30.48" y1="49.53" x2="30.48" y2="39.37" width="0.6096" layer="1"/>
 <wire x1="30.48" y1="39.37" x2="63.5" y2="39.37" width="0.6096" layer="1"/>
-<wire x1="63.5" y1="39.37" x2="64.274" y2="39.584" width="0.6096" layer="1"/>
+<wire x1="63.5" y1="39.37" x2="64.254096875" y2="39.56421875" width="0.6096" layer="1"/>
 </signal>
 <signal name="ENC_1" class="1">
@@
 <wire x1="58.42" y1="41.275" x2="58.42" y2="43.815" width="0.6096" layer="1"/>
 <wire x1="58.42" y1="43.815" x2="62.161" y2="43.815" width="0.6096" layer="1"/>
-<wire x1="62.161" y1="43.815" x2="62.161" y2="44.115" width="0.6096" layer="1"/>
+<wire x1="62.161" y1="43.815" x2="62.141096875" y2="44.09521875" width="0.6096" layer="1"/>
 </signal>
 <signal name="+3.3V">
