File: Electronic/metaPixelFull/UI2/Display.brd (EAGLE design)
At the start: 160 x 100 mm, 34 parts, among them IC1 74HCT14N, IC2 74HCT14N, IC3 74HCT74N, Q1 2N3906

Commit message: Building the UI-Board
Parts:
- moved IC2 31.4 mm to (30.5, 61.0), turned to 180 degrees
- moved IC3 24.1 mm to (19.1, 44.5), turned to 180 degrees
- moved IC1 17.8 mm to (48.3, 49.5)
- moved SV3 8.98 mm to (36.8, 78.7)
- moved Q1 4.58 mm to (54.6, 8.89), turned to 0 degrees
- moved SV1 3.59 mm to (31.8, 11.4)
- moved R1 2.84 mm to (55.9, 3.81), turned to 0 degrees
- moved R2 2.62 mm to (50.8, 14.6), turned to 0 degrees
Routing:
- net +3.3V: track 0.00 -> 86.2 mm, vias 0 -> 4
- net MISO: track 0.00 -> 81.9 mm, vias 0 -> 1
- net MOSI: track 0.00 -> 81.2 mm
- net SCLK: track 0.00 -> 81.0 mm, vias 0 -> 1
- net !MEM_CS: track 0.00 -> 41.2 mm
- net !LCD_CS: track 0.00 -> 39.5 mm, vias 0 -> 1
- net LCD_DC: track 0.00 -> 37.3 mm, vias 0 -> 1
- net GND: track 0.00 -> 36.1 mm, vias 0 -> 1
- net !LCD_RST: track 0.00 -> 32.4 mm
- net BG_LED: track 0.00 -> 15.9 mm
- net N$2: track 0.00 -> 15.9 mm, vias 0 -> 1
- net LCD_LED: track 0.00 -> 10.8 mm
- net KEY_1: track 0.00 -> 6.88 mm
- net KEY_5: track 0.00 -> 6.88 mm
- net KEY_4: track 0.00 -> 6.88 mm
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