File: Electronic/metaPixelFull/UI2/TFT-Display.sch (EAGLE design)
At the start: 34 parts, among them IC1 74HCT14N, IC2 74HCT14N, IC3 74HCT74N, Q1 2N3906

Commit message: Display board layout
Parts:
- HOST: value HOST -> (none)
- renumbered SV1 to HOST, SV3 to KEYBOARD
Connections:
- net ENC_DIR: now also HOST.20; no longer HOST.19
- net ENC_STEP: now also HOST.19; no longer HOST.20
