File: Electronic/metaPixelFull/UI2/TFT-Display.brd (EAGLE design)
At the start: 160 x 100 mm, 34 parts, among them IC1 74HCT14N, IC2 74HCT14N, IC3 74HCT74N, Q1 2N3906

Commit message: Display board layout
Parts:
- removed SV3: (no value), con-harting-ml:ML10L
- added KEYBOARD: (no value), con-harting-ml:ML10L
- HOST: value HOST -> (none)
- moved C10 89.5 mm to (29.2, 24.1), turned to 90 degrees
- moved R18 85.7 mm to (21.6, 43.2), turned to 180 degrees
- moved C1 83.9 mm to (33.0, 36.8), turned to 270 degrees
- moved R3 83.7 mm to (33.0, 44.5), turned to 270 degrees
- moved C2 80.3 mm to (44.5, 34.3), turned to 270 degrees
- moved C7 80.2 mm to (10.8, 52.1), turned to 180 degrees
- moved C3 79.8 mm to (48.3, 36.8), turned to 270 degrees
- moved R14 78.2 mm to (29.2, 47.0), turned to 270 degrees
- moved C9 77.3 mm to (29.2, 39.4), turned to 270 degrees
- moved R7 62.0 mm to (48.3, 44.5), turned to 270 degrees
- moved C8 62.0 mm to (57.1, 24.1), turned to 270 degrees
- moved R20 61.7 mm to (33.0, 24.1), turned to 90 degrees
- moved R17 61.4 mm to (36.8, 41.9), turned to 270 degrees
- moved C6 61.2 mm to (36.8, 34.3), turned to 270 degrees
- moved R4 57.1 mm to (21.6, 48.3), turned to 180 degrees
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- renumbered SV1 to HOST
Connections:
- net +3.3V: now also KEYBOARD.1; no longer SV3.1
- net ENC_1: now also KEYBOARD.7; no longer SV3.7
- net ENC_2: now also KEYBOARD.5; no longer SV3.5
- net ENC_DIR: now also HOST.20; no longer HOST.19
- net ENC_STEP: now also HOST.19; no longer HOST.20
- net GND: now also KEYBOARD.2; no longer SV3.2
- net K_1: now also KEYBOARD.4; no longer SV3.4
- net K_2: now also KEYBOARD.6; no longer SV3.6
- net K_3: now also KEYBOARD.8; no longer SV3.8
- net K_4: now also KEYBOARD.10; no longer SV3.10
- net K_5: now also KEYBOARD.9; no longer SV3.9
Routing:
- net +3.3V: track 86.2 -> 234.4 mm
- net GND: track 36.1 -> 173.5 mm, vias 1 -> 2
- net K1: track 0.00 -> 46.2 mm
- net KEY_4: track 6.88 -> 46.1 mm, vias 0 -> 1
- net KEY_5: track 6.88 -> 43.7 mm, vias 0 -> 1
- net K2: track 0.00 -> 36.1 mm
- net ENC1: track 0.00 -> 30.2 mm
- net ENC_STEP: track 6.88 -> 35.2 mm
- net ENC2: track 0.00 -> 28.3 mm
- net K3: track 0.00 -> 27.2 mm
- net ENC_1: track 0.00 -> 25.0 mm
- net ENC_DIR: track 3.81 -> 25.9 mm
- net K_3: track 0.00 -> 19.6 mm
- net KEY_1: track 6.88 -> 25.9 mm, vias 0 -> 2
- net K_2: track 0.00 -> 18.8 mm
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Other:
- board size 160 x 100 mm -> 68.6 x 63.2 mm

Commit message: The first 3 Boards are ready
Parts:
- moved R6 11.5 mm to (58.4, 34.3)
- moved R8 8.98 mm to (58.4, 39.4)
- moved R10 7.73 mm to (58.4, 43.2)
- moved R14 7.62 mm to (29.2, 39.4)
- moved R9 7.62 mm to (52.1, 39.4)
- moved C4 7.62 mm to (52.1, 31.8)
- moved C9 7.62 mm to (29.2, 31.8)
- moved R18 6.35 mm to (21.6, 49.5)
- moved R4 6.35 mm to (21.6, 41.9)
- moved R15 6.35 mm to (21.6, 44.5)
- moved R3 5.08 mm to (33.0, 39.4)
- moved R7 5.08 mm to (48.3, 39.4)
- moved C1 5.08 mm to (33.0, 31.8)
- moved C3 5.08 mm to (48.3, 31.8)
- moved KEYBOARD 3.81 mm to (40.6, 48.3)
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Routing:
- net +3.3V: track 234.4 -> 220.2 mm
- net GND: track 173.5 -> 184.9 mm
- net K5: track 16.3 -> 8.67 mm
- net K_3: track 19.6 -> 25.9 mm
- net K_5: track 11.2 -> 16.5 mm
- net K4: track 13.2 -> 8.15 mm
- net ENC1: track 30.2 -> 34.9 mm
- net ENC2: track 28.3 -> 32.9 mm
- net K_4: track 11.2 -> 15.2 mm
- net K_1: track 13.8 -> 17.0 mm
- net K_2: track 18.8 -> 21.7 mm
- net ENC_2: track 18.1 -> 20.6 mm
- net K2: track 36.1 -> 34.8 mm
- net K1: track 46.2 -> 45.0 mm
- net ENC_STEP: track 35.2 -> 34.5 mm
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Other:
- board size 68.6 x 63.2 mm -> 67.9 x 58.1 mm

Commit message: minor changes
Parts:
- U$1: value 2.2_TFT_LCD -> 2.2_TFT_LCDNEW; device 2.2"tft:2.2_TFT_LCD -> 2.2"tft:2.2_TFT_LCD_LEDSEE
- moved U$1 33.7 mm to (33.9, 20.3)
Connections:
- net !LCD_CS: now also U$1.P$3_CS; no longer U$1.CS
- net !LCD_RST: now also U$1.P$2_RESET; no longer U$1.RST
- net !MEM_CS: now also U$1.P$2_SD_CS; no longer U$1.SD_CS
- net +3.3V: now also U$1.P$5_VCC; no longer U$1.VCC
- net BG_LED: now also U$1.P$8_LED; no longer U$1.LED
- net GND: now also U$1.P$4_GND; no longer U$1.GND
- net LCD_DC: now also U$1.P$1_DC; no longer U$1.DC
- net MISO: now also U$1.P$3_SD_MISO, U$1.P$9_MISO; no longer U$1.MISO, U$1.SD_MISO
- net MOSI: now also U$1.P$1_SD_MOSI, U$1.P$6_MOSI; no longer U$1.MOSI, U$1.SD_MOSI
- net SCLK: now also U$1.P$4_SD_SCK, U$1.P$7_SCK; no longer U$1.SCK, U$1.SD_SCK
Routing:
- net GND: track 184.9 -> 196.9 mm
- net LCD_DC: track 36.9 -> 36.4 mm
- net BG_LED: track 15.9 -> 16.4 mm
- net !LCD_RST: track 32.4 -> 33.0 mm
- net +3.3V: track 220.2 -> 219.7 mm
Changed lines of the file:
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@@
 <setting verticaltext="up"/>
 </settings>
-<grid distance="0.05" unitdist="inch" unit="inch" style="dots" multiple="1" display="yes" altdistance="0.025" altunitdist="inch" altunit="inch"/>
+<grid distance="0.05" unitdist="inch" unit="inch" style="dots" multiple="1" display="yes" altdistance="0.01" altunitdist="inch" altunit="inch"/>
 <layers>
 <layer number="1" name="Top" color="4" fill="1" visible="yes" active="yes"/>
@@
 <attribute name="VALUE" x="36.8554" y="0" size="1.778" layer="27" ratio="10" rot="R180"/>
 </element>
-<element name="U$1" library="2.2&quot;tft" package="2.2_TFT_LCD" value="2.2_TFT_LCD" x="66.04" y="30.48" rot="MR0"/>
+<element name="U$1" library="2.2&quot;tft" package="2.2_TFT_LCD_LEDSEE" value="2.2_TFT_LCDNEW" x="33.92" y="20.32" rot="MR0"/>
 <element name="C9" library="rcl" package="C025-024X044" value=".1µ" x="29.21" y="31.75" rot="R270"/>
 <element name="R14" library="resistor" package="0204/7" value="15k" x="29.21" y="39.37" rot="R270"/>
@@
 <signal name="GND" class="1">
 <contactref element="HOST" pad="1"/>
-<contactref element="U$1" pad="GND"/>
+<contactref element="U$1" pad="P$4_GND"/>
 <contactref element="IC1" pad="7"/>
 <contactref element="IC2" pad="7"/>
@@
 <wire x1="62.5475" y1="20.6375" x2="62.5475" y2="22.86" width="0.4064" layer="16"/>
 <wire x1="62.5475" y1="22.86" x2="62.5475" y2="27.94" width="0.4064" layer="16"/>
-<wire x1="62.5475" y1="27.94" x2="66.04" y2="27.94" width="0.4064" layer="16"/>
+<wire x1="62.5475" y1="27.94" x2="65.52" y2="27.94" width="0.4064" layer="16"/>
 <wire x1="29.21" y1="25.4" x2="8.89" y2="25.4" width="0.4064" layer="16"/>
 <wire x1="8.89" y1="25.4" x2="8.89" y2="27.94" width="0.4064" layer="16"/>
@@
 <via x="43.18" y="25.4" extent="1-16" drill="0.3048" diameter="0.3048"/>
 <wire x1="43.18" y1="25.4" x2="36.83" y2="25.4" width="0.4064" layer="16"/>
-<wire x1="9.525" y1="52.07" x2="9.525" y2="31.75" width="0.4064" layer="1"/>
-<wire x1="9.525" y1="31.75" x2="8.89" y2="31.75" width="0.4064" layer="1"/>
-<wire x1="8.89" y1="31.75" x2="6.985" y2="31.75" width="0.4064" layer="1"/>
 <wire x1="29.21" y1="30.48" x2="33.02" y2="30.48" width="0.4064" layer="16"/>
 <wire x1="33.02" y1="30.48" x2="36.83" y2="30.48" width="0.4064" layer="16"/>
@@
 <wire x1="36.83" y1="30.48" x2="36.83" y2="27.94" width="0.4064" layer="16"/>
 <wire x1="57.15" y1="22.86" x2="62.5475" y2="22.86" width="0.4064" layer="16"/>
-<wire x1="8.89" y1="27.94" x2="8.89" y2="31.75" width="0.4064" layer="1"/>
+<wire x1="20.955" y1="50.8" x2="10.16" y2="50.8" width="0.4064" layer="1"/>
+<wire x1="10.16" y1="50.8" x2="9.525" y2="50.8" width="0.4064" layer="1"/>
+<wire x1="9.525" y1="50.8" x2="9.525" y2="52.07" width="0.4064" layer="1"/>
+<wire x1="8.89" y1="27.94" x2="10.16" y2="29.21" width="0.4064" layer="1"/>
+<wire x1="10.16" y1="29.21" x2="10.16" y2="31.75" width="0.4064" layer="1"/>
+<wire x1="10.16" y1="31.75" x2="10.16" y2="50.8" width="0.4064" layer="1"/>
+<wire x1="6.985" y1="31.75" x2="10.16" y2="31.75" width="0.4064" layer="1"/>
 </signal>
 <signal name="+5" class="1">
@@
 <signal name="!LCD_CS">
 <contactref element="HOST" pad="7"/>
-<contactref element="U$1" pad="CS"/>
+<contactref element="U$1" pad="P$3_CS"/>
 <wire x1="35.56" y1="12.7" x2="35.56" y2="15.875" width="0.2032" layer="1"/>
 <via x="35.56" y="15.875" extent="1-16" drill="0.3048" diameter="0.254"/>
@@
 <wire x1="58.7375" y1="15.875" x2="64.77" y2="21.59" width="0.2032" layer="16"/>
 <wire x1="64.77" y1="21.59" x2="64.77" y2="24.13" width="0.2032" layer="16"/>
-<wire x1="64.77" y1="24.13" x2="66.04" y2="25.4" width="0.2032" layer="16"/>
+<wire x1="64.77" y1="24.13" x2="65.52" y2="25.4" width="0.2032" layer="16"/>
 </signal>
 <signal name="MISO">
 <contactref element="HOST" pad="9"/>
-<contactref element="U$1" pad="MISO"/>
-<contactref element="U$1" pad="SD_MISO"/>
-<wire x1="2.54" y1="19.05" x2="3.81" y2="19.05" width="0.2032" layer="16"/>
+<contactref element="U$1" pad="P$9_MISO"/>
+<contactref element="U$1" pad="P$3_SD_MISO"/>
+<wire x1="2.32" y1="19.05" x2="3.81" y2="19.05" width="0.2032" layer="16"/>
 <wire x1="3.81" y1="19.05" x2="3.81" y2="7.62" width="0.2032" layer="16"/>
 <wire x1="34.29" y1="11.43" x2="33.02" y2="12.7" width="0.2032" layer="1"/>
@@
 <via x="34.29" y="7.62" extent="1-16" drill="0.3048" diameter="0.254"/>
 <wire x1="34.29" y1="7.62" x2="34.29" y2="11.43" width="0.2032" layer="1"/>
-<wire x1="66.04" y1="10.16" x2="55.5625" y2="10.16" width="0.2032" layer="16"/>
+<wire x1="65.52" y1="10.16" x2="55.5625" y2="10.16" width="0.2032" layer="16"/>
 <wire x1="55.5625" y1="10.16" x2="55.245" y2="9.8425" width="0.2032" layer="16"/>
 <wire x1="55.245" y1="9.8425" x2="53.975" y2="9.8425" width="0.2032" layer="16"/>
@@
 <contactref element="Q1" pad="3"/>
 <contactref element="R1" pad="1"/>
-<contactref element="U$1" pad="VCC"/>
+<contactref element="U$1" pad="P$5_VCC"/>
 <contactref element="KEYBOARD" pad="1"/>
 <contactref element="R20" pad="1"/>
@@
 <wire x1="52.07" y1="3.81" x2="52.07" y2="7.62" width="0.4064" layer="1"/>
 <wire x1="52.07" y1="7.62" x2="53.34" y2="8.89" width="0.4064" layer="1"/>
-<wire x1="66.04" y1="30.48" x2="63.8175" y2="30.48" width="0.4064" layer="1"/>
+<wire x1="65.52" y1="30.48" x2="63.8175" y2="30.48" width="0.4064" layer="1"/>
 <wire x1="63.8175" y1="7.62" x2="52.07" y2="7.62" width="0.4064" layer="16"/>
 <via x="63.8175" y="7.62" extent="1-16" drill="0.3048" diameter="0.254"/>
@@
 <signal name="!LCD_RST">
 <contactref element="HOST" pad="2"/>
-<contactref element="U$1" pad="RST"/>
+<contactref element="U$1" pad="P$2_RESET"/>
 <wire x1="43.18" y1="10.16" x2="48.26" y2="10.16" width="0.2032" layer="16"/>
 <wire x1="48.26" y1="10.16" x2="51.435" y2="13.335" width="0.2032" layer="16"/>
@@
 <wire x1="64.4525" y1="18.7325" x2="66.9925" y2="18.7325" width="0.2032" layer="16"/>
 <wire x1="66.9925" y1="18.7325" x2="66.9925" y2="22.86" width="0.2032" layer="16"/>
-<wire x1="66.9925" y1="22.86" x2="66.04" y2="22.86" width="0.2032" layer="16"/>
+<wire x1="66.9925" y1="22.86" x2="65.52" y2="22.86" width="0.2032" layer="16"/>
 </signal>
 <signal name="MOSI">
 <contactref element="HOST" pad="4"/>
-<contactref element="U$1" pad="MOSI"/>
-<contactref element="U$1" pad="SD_MOSI"/>
-<wire x1="2.54" y1="21.59" x2="5.08" y2="21.59" width="0.2032" layer="16"/>
+<contactref element="U$1" pad="P$6_MOSI"/>
+<contactref element="U$1" pad="P$1_SD_MOSI"/>
+<wire x1="2.32" y1="21.59" x2="5.08" y2="21.59" width="0.2032" layer="16"/>
 <wire x1="5.08" y1="21.59" x2="5.08" y2="8.89" width="0.2032" layer="16"/>
 <wire x1="5.08" y1="8.89" x2="40.64" y2="8.89" width="0.2032" layer="16"/>
 <wire x1="40.64" y1="8.89" x2="48.26" y2="8.89" width="0.2032" layer="16"/>
-<wire x1="66.04" y1="17.78" x2="64.77" y2="17.78" width="0.2032" layer="16"/>
+<wire x1="65.52" y1="17.78" x2="64.77" y2="17.78" width="0.2032" layer="16"/>
 <wire x1="64.77" y1="17.78" x2="59.69" y2="12.7" width="0.2032" layer="16"/>
 <wire x1="59.69" y1="12.7" x2="52.07" y2="12.7" width="0.2032" layer="16"/>
@@
 <signal name="SCLK">
 <contactref element="HOST" pad="6"/>
-<contactref element="U$1" pad="SCK"/>
-<contactref element="U$1" pad="SD_SCK"/>
-<wire x1="2.54" y1="16.51" x2="2.54" y2="6.985" width="0.2032" layer="1"/>
+<contactref element="U$1" pad="P$7_SCK"/>
+<contactref element="U$1" pad="P$4_SD_SCK"/>
 <wire x1="2.54" y1="6.985" x2="38.1" y2="6.985" width="0.2032" layer="1"/>
 <wire x1="38.1" y1="6.985" x2="38.1" y2="8.255" width="0.2032" layer="1"/>
 <wire x1="38.1" y1="8.255" x2="38.1" y2="10.16" width="0.2032" layer="1"/>
-<wire x1="66.04" y1="15.24" x2="64.77" y2="15.24" width="0.2032" layer="16"/>
+<wire x1="65.52" y1="15.24" x2="64.77" y2="15.24" width="0.2032" layer="16"/>
 <wire x1="64.77" y1="15.24" x2="61.595" y2="12.065" width="0.2032" layer="16"/>
 <wire x1="61.595" y1="12.065" x2="52.705" y2="12.065" width="0.2032" layer="16"/>
@@
 <wire x1="48.895" y1="8.255" x2="38.1" y2="8.255" width="0.2032" layer="16"/>
 <via x="38.1" y="8.255" extent="1-16" drill="0.3048" diameter="0.254"/>
+<wire x1="2.32" y1="16.51" x2="2.54" y2="16.002" width="0.2032" layer="1"/>
+<wire x1="2.54" y1="16.002" x2="2.54" y2="6.985" width="0.2032" layer="1"/>
 </signal>
 <signal name="LCD_DC">
 <contactref element="HOST" pad="8"/>
-<contactref element="U$1" pad="DC"/>
+<contactref element="U$1" pad="P$1_DC"/>
 <wire x1="35.56" y1="10.16" x2="36.83" y2="11.43" width="0.2032" layer="1"/>
 <wire x1="36.83" y1="11.43" x2="36.83" y2="15.24" width="0.2032" layer="1"/>
-<wire x1="66.04" y1="20.32" x2="64.135" y2="20.32" width="0.2032" layer="16"/>
+<wire x1="65.52" y1="20.32" x2="64.135" y2="20.32" width="0.2032" layer="16"/>
 <wire x1="64.135" y1="20.32" x2="59.055" y2="15.24" width="0.2032" layer="16"/>
 <wire x1="59.055" y1="15.24" x2="36.83" y2="15.24" width="0.2032" layer="16"/>
@@
 <signal name="!MEM_CS">
 <contactref element="HOST" pad="11"/>
-<contactref element="U$1" pad="SD_CS"/>
-<wire x1="2.54" y1="24.13" x2="6.35" y2="24.13" width="0.2032" layer="16"/>
+<contactref element="U$1" pad="P$2_SD_CS"/>
+<wire x1="2.32" y1="24.13" x2="6.35" y2="24.13" width="0.2032" layer="16"/>
 <wire x1="6.35" y1="24.13" x2="6.35" y2="11.43" width="0.2032" layer="16"/>
 <wire x1="6.35" y1="11.43" x2="29.21" y2="11.43" width="0.2032" layer="16"/>
@@
 </signal>
 <signal name="BG_LED">
-<contactref element="U$1" pad="LED"/>
+<contactref element="U$1" pad="P$8_LED"/>
 <contactref element="Q1" pad="1"/>
-<wire x1="66.04" y1="12.7" x2="66.9925" y2="12.7" width="0.2032" layer="16"/>
+<wire x1="65.52" y1="12.7" x2="66.9925" y2="12.7" width="0.2032" layer="16"/>
 <wire x1="66.9925" y1="12.7" x2="66.9925" y2="8.89" width="0.2032" layer="16"/>
 <wire x1="66.9925" y1="8.89" x2="55.88" y2="8.89" width="0.2032" layer="16"/>

Commit message: adding a couple of data sheets
Routing:
- net +3.3V: track 219.7 -> 218.9 mm
Changed lines of the file:
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@@
 <via x="35.56" y="15.875" extent="1-16" drill="0.3048" diameter="0.254"/>
 <wire x1="35.56" y1="15.875" x2="58.7375" y2="15.875" width="0.2032" layer="16"/>
-<wire x1="58.7375" y1="15.875" x2="64.77" y2="21.59" width="0.2032" layer="16"/>
-<wire x1="64.77" y1="21.59" x2="64.77" y2="24.13" width="0.2032" layer="16"/>
-<wire x1="64.77" y1="24.13" x2="65.52" y2="25.4" width="0.2032" layer="16"/>
+<wire x1="58.7375" y1="15.875" x2="64.262" y2="21.59" width="0.2032" layer="16"/>
+<wire x1="64.262" y1="21.59" x2="64.262" y2="24.384" width="0.2032" layer="16"/>
+<wire x1="64.262" y1="24.384" x2="65.52" y2="25.4" width="0.2032" layer="16"/>
 </signal>
 <signal name="MISO">
@@
 <wire x1="29.21" y1="22.86" x2="26.67" y2="22.86" width="0.4064" layer="1"/>
 <wire x1="26.67" y1="22.86" x2="26.67" y2="29.845" width="0.4064" layer="1"/>
-<wire x1="26.67" y1="29.845" x2="19.05" y2="29.845" width="0.4064" layer="1"/>
-<wire x1="19.05" y1="29.845" x2="19.05" y2="41.91" width="0.4064" layer="1"/>
+<wire x1="26.67" y1="29.845" x2="20.32" y2="29.845" width="0.4064" layer="1"/>
+<wire x1="20.32" y1="29.845" x2="19.05" y2="31.496" width="0.4064" layer="1"/>
+<wire x1="19.05" y1="31.496" x2="19.05" y2="41.91" width="0.4064" layer="1"/>
 <wire x1="33.02" y1="20.32" x2="35.56" y2="22.86" width="0.4064" layer="16"/>
 <wire x1="35.56" y1="22.86" x2="50.8" y2="22.86" width="0.4064" layer="16"/>

Commit message: Reworking the Controller
Parts:
- removed C10: .1µ, rcl:C025-024X044
- removed IC3: 74HCT74N, 74xx-eu:DIL14
- removed R20: 3k3, resistor:0204/7
- moved C7 19.7 mm to (10.8, 32.4)
- moved IC2 17.8 mm to (10.8, 21.6)
- moved R18 8.89 mm to (21.6, 40.6)
- moved R15 6.35 mm to (21.6, 38.1)
- moved R4 6.35 mm to (21.6, 35.6)
- moved R8 5.12 mm to (57.8, 34.3), turned to 270 degrees
- moved R6 4.07 mm to (55.2, 31.8), turned to 270 degrees
- moved R19 3.81 mm to (21.6, 43.2)
- moved R10 3.59 mm to (55.9, 45.7)
Connections:
- removed net ENC_DIR: HOST.20, IC3.5
- removed net ENC_STEP: HOST.19, IC2.12, IC3.3
- removed net N$1: IC2.10, IC3.2
- removed net N$3: IC3.1, IC3.4, R20.2
- new net ENC_A: HOST.19, IC2.10
- new net ENC_B: HOST.20, IC2.12
- net +3.3V: no longer C10.1, IC3.14, R20.1
- net GND: no longer C10.2, IC3.7
Routing:
- net ENC_STEP: track 34.5 -> 0.00 mm
- net ENC_DIR: track 25.9 -> 0.00 mm
- net GND: track 196.9 -> 174.9 mm
- net ENC_B: track 0.00 -> 19.7 mm
- net N$3: track 18.3 -> 0.00 mm
- net +3.3V: track 218.9 -> 202.6 mm, vias 4 -> 6
- net N$1: track 15.9 -> 0.00 mm
- net ENC_A: track 0.00 -> 12.1 mm
- net ENC1: track 34.9 -> 42.5 mm
- net K_2: track 21.7 -> 28.1 mm
- net K_1: track 17.0 -> 21.5 mm
- net K_5: track 16.5 -> 21.0 mm
- net ENC_2: track 20.6 -> 23.4 mm
- net KEY_5: track 43.7 -> 41.2 mm
- net KEY_4: track 46.1 -> 43.7 mm
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