File: Electronic/metaPixelFull/UI2/Cursor-EC60.brd (EAGLE design)
At the start: 40 x 40 mm, 7 parts

Commit message: The first 3 Boards are ready
Routing:
- net KEY_RIGHT: track 7.12 -> 9.27 mm
Changed lines of the file:
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@@
 <contactref element="KEY_RIGHT" pad="P$1"/>
 <contactref element="JP1" pad="2"/>
-<wire x1="34.9724" y1="21.8892" x2="34.7208" y2="21.8892" width="0.762" layer="16"/>
-<wire x1="38.7464" y1="18.1152" x2="34.9724" y2="21.8892" width="0.6096" layer="16"/>
-<wire x1="38.7464" y1="16.983" x2="38.7464" y2="18.1152" width="0.6096" layer="16"/>
-<wire x1="34.7208" y1="21.8892" x2="35.007103125" y2="21.99289375" width="0.6096" layer="16"/>
-<wire x1="38.7464" y1="16.983" x2="38.81" y2="16.92" width="0.762" layer="16"/>
+<wire x1="38.81" y1="16.92" x2="39" y2="16.92" width="0.6096" layer="16"/>
+<wire x1="39" y1="16.92" x2="39" y2="22" width="0.6096" layer="16"/>
+<wire x1="39" y1="22" x2="35.007103125" y2="22" width="0.6096" layer="16"/>
+<wire x1="35.007103125" y1="22" x2="35.007103125" y2="21.99289375" width="0.6096" layer="16"/>
 </signal>
 <signal name="KEY_DOWN" class="1">

Commit message: Fixing the boards
Parts:
- JP1: value (none) -> K1
- JP2: value (none) -> K2
Changed lines of the file:
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@@
 <description>&lt;h1&gt;5 Key cursor cross&lt;/h1&gt;
 &lt;p&gt;circular board which can go inside an ALPS EC60&lt;/p&gt;
-&lt;p&gt;Status: Working&lt;/p&gt;</description>
+&lt;p&gt;Status:
+&lt;ul&gt;
+&lt;li&gt;Working&lt;/li&gt;
+&lt;li&gt;dru ok&lt;/li&gt;
+&lt;/ul&gt;
+&lt;/p&gt;</description>
 <plain>
 <circle x="22.5" y="22" radius="20" width="0.4064" layer="20"/>
@@
 </class>
 </classes>
-<designrules name="default">
-<description language="de">&lt;b&gt;EAGLE Design Rules&lt;/b&gt;
-&lt;p&gt;
-Die Standard-Design-Rules sind so gewählt, dass sie für
-die meisten Anwendungen passen. Sollte ihre Platine
-besondere Anforderungen haben, treffen Sie die erforderlichen
-Einstellungen hier und speichern die Design Rules unter
-einem neuen Namen ab.</description>
-<description language="en">&lt;b&gt;EAGLE Design Rules&lt;/b&gt;
-&lt;p&gt;
-The default Design Rules have been set to cover
-a wide range of applications. Your particular design
-may have different requirements, so please make the
-necessary adjustments and save your customized
-design rules under a new name.</description>
+<designrules name="dirt_cheap_dirty_boards.v1">
+<description language="en">&lt;b&gt;Dirty Cheap Dirty Board Design Rules&lt;/b&gt;
+&lt;br&gt;
+&lt;br&gt;Min width/Spacing: 5/5mil
+&lt;br&gt;Min diameter of finished hole 12mil</description>
 <param name="layerSetup" value="(1*16)"/>
-<param name="mtCopper" value="0.035mm 0.035mm 0.035mm 0.035mm 0.035mm 0.035mm 0.035mm 0.035mm 0.035mm 0.035mm 0.035mm 0.035mm 0.035mm 0.035mm 0.035mm 0.035mm"/>
-<param name="mtIsolate" value="1.5mm 0.15mm 0.2mm 0.15mm 0.2mm 0.15mm 0.2mm 0.15mm 0.2mm 0.15mm 0.2mm 0.15mm 0.2mm 0.15mm 0.2mm"/>
-<param name="mdWireWire" value="8mil"/>
-<param name="mdWirePad" value="8mil"/>
-<param name="mdWireVia" value="8mil"/>
-<param name="mdPadPad" value="8mil"/>
-<param name="mdPadVia" value="8mil"/>
-<param name="mdViaVia" value="8mil"/>
-<param name="mdSmdPad" value="8mil"/>
-<param name="mdSmdVia" value="8mil"/>
-<param name="mdSmdSmd" value="8mil"/>
+<param name="mtCopper" value="0.035mm 0.0175mm 0.035mm 0.035mm 0.035mm 0.035mm 0.035mm 0.035mm 0.035mm 0.035mm 0.035mm 0.035mm 0.035mm 0.035mm 0.0175mm 0.035mm"/>
+<param name="mtIsolate" value="1.5mm 1.1mm 0.2mm 0.15mm 0.2mm 0.15mm 0.2mm 0.15mm 0.2mm 0.15mm 0.2mm 0.15mm 0.2mm 0.15mm 0.2mm"/>
+<param name="mdWireWire" value="5mil"/>
+<param name="mdWirePad" value="5mil"/>
+<param name="mdWireVia" value="5mil"/>
+<param name="mdPadPad" value="5mil"/>
+<param name="mdPadVia" value="5mil"/>
+<param name="mdViaVia" value="5mil"/>
+<param name="mdSmdPad" value="0mil"/>
+<param name="mdSmdVia" value="0mil"/>
+<param name="mdSmdSmd" value="0mil"/>
 <param name="mdViaViaSameLayer" value="8mil"/>
 <param name="mnLayersViaInSmd" value="2"/>
-<param name="mdCopperDimension" value="40mil"/>
-<param name="mdDrill" value="8mil"/>
+<param name="mdCopperDimension" value="10mil"/>
+<param name="mdDrill" value="10mil"/>
 <param name="mdSmdStop" value="0mil"/>
-<param name="msWidth" value="10mil"/>
-<param name="msDrill" value="24mil"/>
-<param name="msMicroVia" value="9.99mm"/>
+<param name="msWidth" value="5mil"/>
+<param name="msDrill" value="12mil"/>
+<param name="msMicroVia" value="12mil"/>
 <param name="msBlindViaRatio" value="0.5"/>
 <param name="rvPadTop" value="0.25"/>
@@
 <param name="rlMinPadBottom" value="10mil"/>
 <param name="rlMaxPadBottom" value="20mil"/>
-<param name="rlMinViaOuter" value="8mil"/>
+<param name="rlMinViaOuter" value="6mil"/>
 <param name="rlMaxViaOuter" value="20mil"/>
-<param name="rlMinViaInner" value="8mil"/>
+<param name="rlMinViaInner" value="6mil"/>
 <param name="rlMaxViaInner" value="20mil"/>
 <param name="rlMinMicroViaOuter" value="4mil"/>
@@
 <param name="psTop" value="-1"/>
 <param name="psBottom" value="-1"/>
-<param name="psFirst" value="-1"/>
+<param name="psFirst" value="0"/>
 <param name="psElongationLong" value="100"/>
 <param name="psElongationOffset" value="100"/>
 <param name="mvStopFrame" value="1"/>
 <param name="mvCreamFrame" value="0"/>
-<param name="mlMinStopFrame" value="4mil"/>
-<param name="mlMaxStopFrame" value="4mil"/>
+<param name="mlMinStopFrame" value="2mil"/>
+<param name="mlMaxStopFrame" value="2mil"/>
 <param name="mlMinCreamFrame" value="0mil"/>
 <param name="mlMaxCreamFrame" value="0mil"/>
-<param name="mlViaStopLimit" value="0mil"/>
+<param name="mlViaStopLimit" value="25mil"/>
 <param name="srRoundness" value="0"/>
 <param name="srMinRoundness" value="0mil"/>
@@
 <param name="checkAngle" value="0"/>
 <param name="checkFont" value="1"/>
-<param name="checkRestrict" value="1"/>
+<param name="checkRestrict" value="0"/>
 <param name="useDiameter" value="13"/>
 <param name="maxErrors" value="50"/>
@@
 <attribute name="NAME" x="22.5" y="40.5" size="1.27" layer="21" rot="R180" align="bottom-center"/>
 </element>
-<element name="JP1" library="pinhead" package="1X03" value="" x="35.007103125" y="21.99289375" rot="MR270"/>
-<element name="JP2" library="pinhead" package="1X03" value="" x="10" y="22" rot="MR90"/>
+<element name="JP1" library="pinhead" package="1X03" value="K1" x="35.007103125" y="21.99289375" rot="MR270"/>
+<element name="JP2" library="pinhead" package="1X03" value="K2" x="10" y="22" rot="MR90"/>
 </elements>
 <signals>
