File: Electronic/metaPixelFull/UI2/Cursor-EC60.sch (EAGLE design)
At the start: 7 parts

Commit message: Fixing the boards
Parts:
- JP1: value (none) -> K1
- JP2: value (none) -> K2
Other:
- note added: "Cursor Keypad build insidean ALPS EC60A/B"
- note removed: "Cursor Keypad for usage inside an ALPS EC60A/B"
Changed lines of the file:
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@@
 </classes>
 <parts>
-<part name="FRAME2" library="frames" deviceset="A4L-LOC" device=""/>
+<part name="FRAME2" library="frames" deviceset="A4L-LOC" device="" value="Cursor Pad"/>
 <part name="KEY_LEFT" library="mec switches" deviceset="3FT1D" device=""/>
 <part name="GND2" library="supply1" deviceset="GND" device=""/>
@@
 <part name="KEY_UP" library="mec switches" deviceset="3FT1D" device=""/>
 <part name="GND5" library="supply1" deviceset="GND" device=""/>
-<part name="JP1" library="pinhead" deviceset="PINHD-1X3" device=""/>
-<part name="JP2" library="pinhead" deviceset="PINHD-1X3" device=""/>
+<part name="JP1" library="pinhead" deviceset="PINHD-1X3" device="" value="K1"/>
+<part name="JP2" library="pinhead" deviceset="PINHD-1X3" device="" value="K2"/>
 </parts>
 <sheets>
@@
 <description>&lt;h1&gt;Cursor Keypad&lt;/h1&gt;</description>
 <plain>
-<text x="162.56" y="22.86" size="2.54" layer="94" align="top-left">Cursor Keypad for usage inside
-an ALPS EC60A/B</text>
+<text x="162.56" y="22.86" size="2.54" layer="94" align="top-left">Cursor Keypad build
+insidean ALPS EC60A/B</text>
 </plain>
 <instances>
@@
 </sheet>
 </sheets>
-<errors>
-</errors>
 </schematic>
 </drawing>
