File: Electronic/metaPixelFull/UI2/Debouncer.brd (EAGLE design)
At the start: 56 x 60 mm, 28 parts, among them IC1 74HCT14N, IC2 74HCT14N

Commit message: Fixing the boards
Parts:
- SK3: value (none) -> Keyboard
- moved C8 1.27 mm to (8.89, 29.2), turned to 0 degrees
Routing:
- net +3.3V: track 0.00 -> 154.5 mm
- net GND: track 0.00 -> 129.0 mm
- net K5: track 0.00 -> 33.8 mm
- net K1: track 0.00 -> 33.1 mm
- net K2: track 0.00 -> 27.4 mm
- net K4: track 0.00 -> 27.3 mm
- net K3: track 0.00 -> 26.2 mm
- net K_4: track 0.00 -> 25.7 mm
- net ENC1: track 0.00 -> 25.3 mm
- net !LCD_CS: track 0.00 -> 21.4 mm
- net MISO: track 0.00 -> 21.4 mm
- net SCLK: track 0.00 -> 21.4 mm
- net LCD_DC: track 0.00 -> 21.4 mm
- net K_3: track 0.00 -> 20.9 mm
- net KEY_3: track 0.00 -> 20.5 mm
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