File: Electronic/metaPixelFull/UI2/Debouncer.sch (EAGLE design)
At the start: 31 parts, among them IC1 74HCT14N, IC2 74HCT14N, Q1 2N3906

Commit message: Removing the TFT from the Debouncer
Parts:
- removed U$1: 2.2_TFT_LCDNEW, 2.2"tft:2.2_TFT_LCDNEW
- added X1: MICS-14, con-lumberg:MICS-14
Connections:
- net !LCD_CS: no longer U$1.CS
- net !LCD_RST: no longer U$1.RST
- net !MEM_CS: no longer U$1.SD_CS
- net +3.3V: no longer U$1.VCC
- net BG_LED: no longer U$1.LED
- net GND: no longer U$1.GND
- net LCD_DC: no longer U$1.DC
- net MISO: no longer U$1.MISO, U$1.SD_MISO
- net MOSI: no longer U$1.MOSI, U$1.SD_MOSI
- net SCLK: no longer U$1.SCK, U$1.SD_SCK
Changed lines of the file:
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@@
 <part name="FRAME1" library="frames" deviceset="A4L-LOC" device=""/>
 <part name="FRAME2" library="frames" deviceset="A4L-LOC" device=""/>
-<part name="U$1" library="2.2&quot;tft" deviceset="2.2_TFT_LCD" device="NEW" value="2.2_TFT_LCDNEW"/>
 <part name="C9" library="rcl" deviceset="C-EU" device="025-024X044" value=".1µ"/>
 <part name="R14" library="resistor" deviceset="R-EU_" device="0204/7" value="15k"/>
@@
 <part name="C7" library="rcl" deviceset="C-EU" device="025-024X044" value=".1µ"/>
 <part name="C8" library="rcl" deviceset="C-EU" device="025-024X044" value=".1µ"/>
+<part name="X1" library="con-lumberg" deviceset="MICS-14" device=""/>
 </parts>
 <sheets>
@@
 <instance part="FRAME1" gate="G$1" x="0" y="0"/>
 <instance part="FRAME2" gate="G$1" x="0" y="0"/>
-<instance part="U$1" gate="G$1" x="132.08" y="132.08"/>
+<instance part="X1" gate="G$1" x="132.08" y="137.16" rot="MR0"/>
 </instances>
 <busses>
@@
 <segment>
 <wire x1="93.98" y1="139.7" x2="111.76" y2="139.7" width="0.1524" layer="91"/>
-<pinref part="U$1" gate="G$1" pin="GND"/>
 <label x="93.98" y="139.7" size="1.27" layer="95" rot="R180" xref="yes"/>
 </segment>
@@
 <wire x1="111.76" y1="137.16" x2="93.98" y2="137.16" width="0.1524" layer="91"/>
 <label x="93.98" y="137.16" size="1.27" layer="95" rot="R180" xref="yes"/>
-<pinref part="U$1" gate="G$1" pin="CS"/>
 </segment>
 </net>
@@
 <wire x1="111.76" y1="121.92" x2="93.98" y2="121.92" width="0.1524" layer="91"/>
 <label x="93.98" y="121.92" size="1.27" layer="95" rot="R180" xref="yes"/>
-<pinref part="U$1" gate="G$1" pin="MISO"/>
-</segment>
-<segment>
-<wire x1="152.4" y1="130.81" x2="165.1" y2="130.81" width="0.1524" layer="91"/>
-<label x="165.1" y="130.81" size="1.27" layer="95" xref="yes"/>
-<pinref part="U$1" gate="G$1" pin="SD_MISO"/>
+</segment>
+<segment>
+<wire x1="106.68" y1="148.59" x2="93.98" y2="148.59" width="0.1524" layer="91"/>
+<label x="93.98" y="148.59" size="1.27" layer="95" rot="MR0" xref="yes"/>
 </segment>
 </net>
@@
 </segment>
 <segment>
-<pinref part="U$1" gate="G$1" pin="VCC"/>
 <wire x1="111.76" y1="142.24" x2="93.98" y2="142.24" width="0.1524" layer="91"/>
 <label x="93.98" y="142.24" size="1.27" layer="95" rot="R180" xref="yes"/>
@@
 <wire x1="93.98" y1="134.62" x2="111.76" y2="134.62" width="0.1524" layer="91"/>
 <label x="93.98" y="134.62" size="1.27" layer="95" rot="R180" xref="yes"/>
-<pinref part="U$1" gate="G$1" pin="RST"/>
 </segment>
 </net>
@@
 <wire x1="93.98" y1="129.54" x2="111.76" y2="129.54" width="0.1524" layer="91"/>
 <label x="93.98" y="129.54" size="1.27" layer="95" rot="R180" xref="yes"/>
-<pinref part="U$1" gate="G$1" pin="MOSI"/>
-</segment>
-<segment>
-<wire x1="152.4" y1="133.35" x2="165.1" y2="133.35" width="0.1524" layer="91"/>
-<label x="165.1" y="133.35" size="1.27" layer="95" xref="yes"/>
-<pinref part="U$1" gate="G$1" pin="SD_MOSI"/>
+</segment>
+<segment>
+<wire x1="106.68" y1="151.13" x2="93.98" y2="151.13" width="0.1524" layer="91"/>
+<label x="93.98" y="151.13" size="1.27" layer="95" rot="MR0" xref="yes"/>
 </segment>
 </net>
@@
 <wire x1="111.76" y1="127" x2="93.98" y2="127" width="0.1524" layer="91"/>
 <label x="93.98" y="127" size="1.27" layer="95" rot="R180" xref="yes"/>
-<pinref part="U$1" gate="G$1" pin="SCK"/>
-</segment>
-<segment>
-<wire x1="152.4" y1="128.27" x2="165.1" y2="128.27" width="0.1524" layer="91"/>
-<label x="165.1" y="128.27" size="1.27" layer="95" xref="yes"/>
-<pinref part="U$1" gate="G$1" pin="SD_SCK"/>
+</segment>
+<segment>
+<wire x1="106.68" y1="146.05" x2="93.98" y2="146.05" width="0.1524" layer="91"/>
+<label x="93.98" y="146.05" size="1.27" layer="95" rot="MR0" xref="yes"/>
 </segment>
 </net>
@@
 <wire x1="111.76" y1="132.08" x2="93.98" y2="132.08" width="0.1524" layer="91"/>
 <label x="93.98" y="132.08" size="1.27" layer="95" rot="R180" xref="yes"/>
-<pinref part="U$1" gate="G$1" pin="DC"/>
 </segment>
 </net>
@@
 </segment>
 <segment>
-<wire x1="152.4" y1="135.89" x2="165.1" y2="135.89" width="0.1524" layer="91"/>
-<label x="165.1" y="135.89" size="1.27" layer="95" xref="yes"/>
-<pinref part="U$1" gate="G$1" pin="SD_CS"/>
+<wire x1="106.68" y1="153.67" x2="93.98" y2="153.67" width="0.1524" layer="91"/>
+<label x="93.98" y="153.67" size="1.27" layer="95" rot="MR0" xref="yes"/>
 </segment>
 </net>
@@
 <wire x1="93.98" y1="124.46" x2="111.76" y2="124.46" width="0.1524" layer="91"/>
 <label x="93.98" y="124.46" size="1.27" layer="95" rot="R180" xref="yes"/>
-<pinref part="U$1" gate="G$1" pin="LED"/>
-</segment>
-<segment>
+</segment>
+<segment>

Commit message: rework UI
Parts:
- removed HOST: (no value), con-harting-ml:ML20L
- removed KEYBOARD: (no value), con-harting-ml:ML10L
- removed Q1: 2N3906, transistor-pnp:2N3906
- removed R1: 10k, resistor:R-EU_0204/7
- removed R2: 100, resistor:R-EU_0204/7
- removed X1: MICS-14, con-lumberg:MICS-14
- added SK1: Host, jt-con-micromatch:MMATCH-20-PTH
- added SK2: Display, jt-con-micromatch:MMATCH-10-PTH
- added SK3: (no value), jt-con-micromatch:MMATCH-10-PTH
Connections:
- removed net +5: HOST.3
- removed net BG_LED: Q1.C
- removed net N$19: HOST.15
- removed net N$2: Q1.B, R1.2, R2.2
- removed net N$20: HOST.17
- net !LCD_CS: now also SK1.6, SK2.3; no longer HOST.7
- net !LCD_RST: now also SK1.7, SK2.4; no longer HOST.2
- net !MEM_CS: now also SK1.13, SK2.10; no longer HOST.11
- net +3.3V: now also SK1.17, SK1.19, SK2.1, SK3.9; no longer HOST.13, KEYBOARD.1, Q1.E, R1.1
- net ENC_1: now also SK3.4; no longer KEYBOARD.7
- net ENC_2: now also SK3.1; no longer KEYBOARD.5
- net ENC_A: now also SK1.14; no longer HOST.19
- net ENC_B: now also SK1.15; no longer HOST.20
- net GND: now also SK1.16, SK1.18, SK1.20, SK2.2, SK3.2; no longer HOST.1, KEYBOARD.2
- net K1: now also IC1C.I; no longer IC1A.I
- net K3: now also IC1A.I; no longer IC1C.I
- net K5: now also IC1F.I; no longer IC1D.I
- net KEY_1: now also IC1C.O, SK1.1; no longer HOST.10, IC1A.O
- net KEY_2: now also SK1.2; no longer HOST.12
- net KEY_3: now also IC1A.O, SK1.3; no longer HOST.14, IC1C.O
- net KEY_4: now also IC1F.O, SK1.4; no longer HOST.16, IC1D.O
- net KEY_5: now also SK1.5; no longer HOST.18
- net K_1: now also SK3.10; no longer KEYBOARD.4
- net K_2: now also SK3.7; no longer KEYBOARD.6
- net K_3: now also SK3.8; no longer KEYBOARD.8
- net K_4: now also SK3.6; no longer KEYBOARD.10
- net K_5: now also SK3.3; no longer KEYBOARD.9
- net LCD_DC: now also SK1.8, SK2.5; no longer HOST.8
- net LCD_LED: now also SK1.11, SK2.8; no longer HOST.5, R2.1
- net MISO: now also SK1.12, SK2.9; no longer HOST.9
- net MOSI: now also SK1.9, SK2.6; no longer HOST.4
- net SCLK: now also SK1.10, SK2.7; no longer HOST.6

Commit message: Fixing the boards
Parts:
- SK3: value (none) -> Keyboard
Changed lines of the file:
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@@
 &lt;p&gt;4 channel switch debouncer and encoder signal conditioning.&lt;/p&gt;
 &lt;p&gt;SPI for connecting a 2.2" TFT and memory card reader&lt;/p&gt;
-&lt;p&gt;Status: Rework finished&lt;/p&gt;</description>
+&lt;p&gt;Status:
+&lt;ul&gt;
+&lt;li&gt;Rework finished&lt;/li&gt;
+&lt;li&gt;Placement final&lt;/li&gt;
+&lt;li&gt;Routing finished&lt;li&gt;
+&lt;/ul&gt;
+&lt;/p&gt;</description>
 <attributes>
 </attributes>
@@
 </classes>
 <parts>
-<part name="FRAME1" library="frames" deviceset="A4L-LOC" device=""/>
-<part name="FRAME2" library="frames" deviceset="A4L-LOC" device=""/>
+<part name="FRAME2" library="frames" deviceset="A4L-LOC" device="" value="Connectors"/>
 <part name="C9" library="rcl" deviceset="C-EU" device="025-024X044" value=".1µ"/>
 <part name="R14" library="resistor" deviceset="R-EU_" device="0204/7" value="15k"/>
@@
 <part name="R10" library="resistor" deviceset="R-EU_" device="0204/7" value="82k"/>
 <part name="IC1" library="74xx-eu" deviceset="74*14" device="N" technology="HCT"/>
-<part name="FRAME3" library="frames" deviceset="A3L-LOC" device=""/>
+<part name="FRAME3" library="frames" deviceset="A3L-LOC" device="" value="Debounce"/>
 <part name="R16" library="resistor" deviceset="R-EU_" device="0204/7" value="10k"/>
 <part name="R17" library="resistor" deviceset="R-EU_" device="0204/7" value="10k"/>
@@
 <part name="SK1" library="jt-con-micromatch" deviceset="MMATCH-20-*" device="PTH" value="Host"/>
 <part name="SK2" library="jt-con-micromatch" deviceset="MMATCH-10-*" device="PTH" value="Display"/>
-<part name="SK3" library="jt-con-micromatch" deviceset="MMATCH-10-*" device="PTH"/>
+<part name="SK3" library="jt-con-micromatch" deviceset="MMATCH-10-*" device="PTH" value="Keyboard"/>
 </parts>
 <sheets>
 <sheet>
+<description>&lt;H1&gt;Babelfisch&lt;/h1&gt;
+&lt;p&gt; in tüten&lt;/p&gt;</description>
 <plain>
 </plain>
 <instances>
-<instance part="FRAME1" gate="G$1" x="0" y="0"/>
 <instance part="FRAME2" gate="G$1" x="0" y="0"/>
 <instance part="SK1" gate="G$1" x="53.34" y="106.68"/>
