File: Electronic/metaPixelFull/UI2/EC60_1.brd (EAGLE design)
At the start: 66 x 65.7 mm, 4 parts

Commit message: Building the UI-Board
Other:
- board size 66 x 65.7 mm -> 66 x 66 mm
Changed lines of the file:
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@@
 <setting verticaltext="up"/>
 </settings>
-<grid distance="0.1" unitdist="inch" unit="mil" style="lines" multiple="1" display="yes" altdistance="0.05" altunitdist="inch" altunit="mil"/>
+<grid distance="1" unitdist="mm" unit="mm" style="lines" multiple="1" display="yes" altdistance="0.1" altunitdist="mm" altunit="mm"/>
 <layers>
 <layer number="1" name="Top" color="4" fill="1" visible="yes" active="yes"/>
@@
 <plain>
 <wire x1="0" y1="0" x2="66.02" y2="0" width="0" layer="20"/>
-<wire x1="66.02" y1="0" x2="66.02" y2="65.71" width="0" layer="20"/>
-<wire x1="66.02" y1="65.71" x2="0" y2="65.71" width="0" layer="20"/>
-<wire x1="0" y1="65.71" x2="0" y2="0" width="0" layer="20"/>
+<wire x1="66.02" y1="0" x2="66.02" y2="66.01" width="0" layer="20"/>
+<wire x1="66.02" y1="66.01" x2="0" y2="65.97" width="0" layer="20"/>
+<wire x1="0" y1="65.97" x2="0" y2="0" width="0" layer="20"/>
 <hole x="22.52" y="46.02" drill="3.2"/>
 <hole x="43.52" y="46.02" drill="3.2"/>

Commit message: The first 3 Boards are ready
Changed lines of the file:
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@@
 <hole x="22.52" y="20.02" drill="3.2"/>
 <hole x="43.52" y="20.02" drill="3.2"/>
-<hole x="6.02" y="60.02" drill="3.2"/>
-<hole x="60.02" y="60.02" drill="3.2"/>
-<hole x="6.02" y="6.02" drill="3.2"/>
-<hole x="60.02" y="6.02" drill="3.2"/>
+<hole x="5.02" y="61.02" drill="3.2"/>
+<hole x="61.02" y="61.02" drill="3.2"/>
+<hole x="5.02" y="4.02" drill="3.2"/>
+<hole x="61.02" y="4.02" drill="3.2"/>
 <text x="45.72" y="22.86" size="1.778" layer="25" rot="R90" align="center-left">GND</text>
 <text x="25.4" y="27.94" size="1.778" layer="25" rot="R180" align="center-left">Center</text>
@@
 <wire x1="63.198096875" y1="41.82921875" x2="55.88" y2="41.82921875" width="0.6096" layer="16"/>
 <wire x1="55.88" y1="41.82921875" x2="36.91078125" y2="41.82921875" width="0.6096" layer="16"/>
-<wire x1="36.91078125" y1="41.82921875" x2="36.83" y2="41.91" width="0.4064" layer="16"/>
 <wire x1="36.83" y1="41.91" x2="36.83" y2="50.8" width="0.6096" layer="16"/>
 <wire x1="36.83" y1="50.8" x2="38.1" y2="52.07" width="0.6096" layer="16"/>
 <wire x1="45.5113375" y1="30.46031875" x2="55.86031875" y2="30.46031875" width="0.6096" layer="16"/>
-<wire x1="55.86031875" y1="30.46031875" x2="55.88" y2="30.48" width="0.4064" layer="16"/>
 <wire x1="55.88" y1="30.48" x2="55.88" y2="41.82921875" width="0.6096" layer="16"/>
+<wire x1="55.86031875" y1="30.46031875" x2="55.88" y2="30.48" width="0" layer="19" extent="16-16"/>
+<wire x1="36.83" y1="41.91" x2="36.91078125" y2="41.82921875" width="0" layer="19" extent="16-16"/>
 </signal>
 <signal name="K_1" class="1">
 <contactref element="SV1" pad="4"/>
 <contactref element="JP1" pad="2"/>
-<wire x1="45.5113375" y1="33.00031875" x2="46.97031875" y2="33.00031875" width="0.4064" layer="16"/>
+<wire x1="45.5113375" y1="33.00031875" x2="46.97031875" y2="33.00031875" width="0.6096" layer="16"/>
 <wire x1="46.97031875" y1="33.00031875" x2="48.26" y2="33.02" width="0.6096" layer="16"/>
 <wire x1="48.26" y1="33.02" x2="48.26" y2="38.1" width="0.6096" layer="16"/>

Commit message: Fixing the boards
Parts:
- removed SV1: (no value), con-harting-ml:ML10L
- added SK1: Keys, jt-con-micromatch:AMP-215079-10
- JP1: value (none) -> K1
- JP2: value (none) -> K2
Connections:
- net +3.3V: now also SK1.9; no longer SV1.1
- net ENC_1: now also SK1.4; no longer SV1.5
- net ENC_2: now also SK1.1; no longer SV1.7
- net GND: now also SK1.2; no longer SV1.2
- net K_1: now also SK1.10; no longer SV1.4
- net K_2: now also SK1.7; no longer SV1.6
- net K_3: now also SK1.8; no longer SV1.8
- net K_4: now also SK1.6; no longer SV1.10
- net K_5: now also SK1.3; no longer SV1.9
Routing:
- net GND: track 58.7 -> 51.4 mm
- net K_2: track 30.8 -> 24.0 mm
- net K_1: track 36.3 -> 30.7 mm
- net ENC_2: track 44.0 -> 39.5 mm
- net K_5: track 26.5 -> 29.8 mm
- net ENC_1: track 40.2 -> 37.8 mm
- net K_4: track 25.8 -> 28.2 mm
- net K_3: track 25.8 -> 24.6 mm
