File: Electronic/metaPixelFull/UI2/EC60_1.sch (EAGLE design)
At the start: 4 parts

Commit message: Fixing the boards
Parts:
- removed SV1: (no value), con-harting-ml:ML10L
- added SK1: Keys, jt-con-micromatch:MMATCH-10-PTH
- JP1: value (none) -> K1
- JP2: value (none) -> K2
Connections:
- net +3.3V: now also SK1.9; no longer SV1.1
- net ENC_1: now also SK1.4; no longer SV1.5
- net ENC_2: now also SK1.1; no longer SV1.7
- net GND: now also SK1.2; no longer SV1.2
- net K_1: now also SK1.10; no longer SV1.4
- net K_2: now also SK1.7; no longer SV1.6
- net K_3: now also SK1.8; no longer SV1.8
- net K_4: now also SK1.6; no longer SV1.10
- net K_5: now also SK1.3; no longer SV1.9
Other:
- moved on the sheet: JP1, JP2
