File: Electronic/metaPixelFull/UI2/TFT-Board.sch (EAGLE design)
At the start: 5 parts, among them Q1 2N3906

Commit message: Fixing the boards
Parts:
- R1: value (none) -> 100
- R2: value (none) -> 10k
- SK1: value (none) -> SPI
Changed lines of the file:
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@@
 <setting verticaltext="up"/>
 </settings>
-<grid distance="0.1" unitdist="inch" unit="inch" style="lines" multiple="1" display="no" altdistance="0.05" altunitdist="inch" altunit="inch"/>
+<grid distance="0.1" unitdist="inch" unit="inch" style="lines" multiple="1" display="no" altdistance="0.01" altunitdist="inch" altunit="inch"/>
 <layers>
 <layer number="1" name="Top" color="4" fill="1" visible="no" active="no"/>
@@
 </layers>
 <schematic xreflabel="%F%N/%S.%C%R" xrefpart="/%S.%C%R">
+<description>&lt;h1&gt;TFT adaptor board&lt;/h1&gt;
+&lt;p&gt;simple adaptor from microMaTch 10 to Ledsee 2.2" TFT.&lt;/p&gt;
+&lt;p&gt;Status:
+&lt;ul&gt;
+&lt;li&gt;Placement final&lt;/li&gt;
+&lt;li&gt;Routing finished&lt;li&gt;
+&lt;/ul&gt;
+&lt;/p&gt;</description>
 <attributes>
 </attributes>
@@
 </variantdefs>
 <classes>
-<class number="0" name="default" width="0" drill="0">
+<class number="0" name="default" width="0.2032" drill="0">
+</class>
+<class number="1" name="SUPPLY" width="0.4064" drill="0">
 </class>
 </classes>
 <parts>
-<part name="FRAME1" library="frames" deviceset="A3L-LOC" device=""/>
+<part name="FRAME1" library="frames" deviceset="A3L-LOC" device="" value="TFT Board"/>
 <part name="U$1" library="2.2&quot;tft" deviceset="2.2_TFT_LCD" device="NEW"/>
 <part name="Q1" library="transistor-pnp" deviceset="2N3906" device=""/>
-<part name="R1" library="resistor" deviceset="R-EU_" device="0204/7"/>
-<part name="R2" library="resistor" deviceset="R-EU_" device="0204/7"/>
-<part name="SK1" library="jt-con-micromatch" deviceset="MMATCH-10-*" device="PTH"/>
+<part name="R1" library="resistor" deviceset="R-EU_" device="0204/7" value="100"/>
+<part name="R2" library="resistor" deviceset="R-EU_" device="0204/7" value="10k"/>
+<part name="SK1" library="jt-con-micromatch" deviceset="MMATCH-10-*" device="PTH" value="SPI"/>
 </parts>
 <sheets>
@@
 </segment>
 </net>
-<net name="+3.3V" class="0">
+<net name="+3.3V" class="1">
 <segment>
 <pinref part="R2" gate="G$1" pin="1"/>
@@
 </segment>
 </net>
-<net name="GND" class="0">
+<net name="GND" class="1">
 <segment>
 <pinref part="U$1" gate="G$1" pin="GND"/>
@@
 </sheet>
 </sheets>
+<errors>
+</errors>
 </schematic>
 </drawing>
